File: LoRaNode.sch (KiCad schematic (older format))
At the start: 33 parts, among them J1 Conn_01x09, J2 Conn_01x03, J3 ISP, J4 D2, J5 D3, J6 Conn_01x06, J7 Conn_01x01, J8 Conn_01x01, SW1 SW_Push, U1 RFM95W-868S2, U2 ATMEGA328P-AU, Y1 8MHz HC5032/4

Commit message: changes for balloon baord
Parts:
- added R?: 10k, Resistor_SMD:R_0603_1608Metric, symbol device:R
- added U?: DHT11, SNR4-2.54-25.0X15.0X7.0MM, symbol TEM-HUM-AM2302_4P-25.0X15.0MM_:TEM-HUM-AM2302(4P-25.0X15.0MM)
- J7, J8: symbol Connector:Conn_01x01 -> LoRaNode-rescue:Conn_01x01-Connector
- SW1: symbol Switch:SW_Push -> LoRaNode-rescue:SW_Push-Switch
Connections:
- wire segments 117 -> 131
Other:
- moved on the sheet: C1, C10, C11, C12, C2, C3, C4, C5, C6, C7, C8, C9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
