File: _saved_LoRaNode.sch (KiCad schematic (older format))
At the start: 31 parts, among them J1 Conn_01x09, J2 Conn_01x03, J4 ISP, J5 Conn_01x06, J8 D2, J9 D3, SW1 SW_Push, U1 RFM95W-868S2, U4 ATMEGA328P-AU, Y1 8MHz HC5032/4

Commit message: changes for balloon baord
Parts:
- added J7, J8: Conn_01x01, MountingHole:MountingHole_2.2mm_M2, symbol LoRaNode-rescue:Conn_01x01-Connector
- added J?: CONN_01X04_BMP, symbol LoRaNode-rescue:CONN_01X04-RESCUE-Arduino_Mini-Arduino_Mini-rescue
- added R?: 10k, Resistor_SMD:R_0603_1608Metric, symbol device:R
- added U?: DHT11, SNR4-2.54-25.0X15.0X7.0MM, symbol TEM-HUM-AM2302_4P-25.0X15.0MM_:TEM-HUM-AM2302(4P-25.0X15.0MM)
- J1: symbol Connector:Conn_01x09 -> LoRaNode-rescue:Conn_01x09-Connector
- J2: symbol Connector:Conn_01x03 -> LoRaNode-rescue:Conn_01x03-Connector
- J3: renamed from J4; symbol Connector:Conn_02x03_Odd_Even -> LoRaNode-rescue:Conn_02x03_Odd_Even-Connector
- J4: renamed from J8; symbol Connector:Conn_01x01 -> LoRaNode-rescue:Conn_01x01-Connector
- J5: renamed from J9; symbol Connector:Conn_01x01 -> LoRaNode-rescue:Conn_01x01-Connector
- J6: renamed from J5; symbol Connector:Conn_01x06 -> LoRaNode-rescue:Conn_01x06-Connector
- SW1: symbol Switch:SW_Push -> LoRaNode-rescue:SW_Push-Switch
- U1: footprint footprints:RFM95W -> MYLIB:HOPERF_RFM95W_SMD
- U2: renamed from U4; symbol atmel:ATMEGA328P-AU -> LoRaNode-rescue:ATMEGA328P-AU-atmel
- Y1: symbol device:Crystal_GND24_Small -> LoRaNode-rescue:Crystal_GND24_Small-device
- renumbered C11 to C1, C17 to C10, C18 to C11, C19 to C12, C13 to C2, C1 to C3, C2 to C4, C20 to C5, C12 to C6, C14 to C7, C15 to C8, C16 to C9, R14 to R1, R15 to R2, R2 to R3, R1 to R4, R16 to R5, R17 to R6, R13 to R7
Connections:
- wire segments 117 -> 137
- no-connect marks 3 -> 5
Other:
- moved on the sheet: C1, C10, C11, C12, C2, C3, C4, C5, C6, C7, C8, C9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
